Commit message: Rebase from 'upstream'

File: pal_robotiq_description/urdf/robotiq.ros2_control.xacro (robot description, xacro)
@@ -13,4 +13,12 @@
  -->
 <robot xmlns:xacro="http://ros.org/wiki/xacro">
+    <xacro:macro name="ros2_control_mimic_joint" params="mimic_joint_name actuated_joint_name multiplier" >
+      <joint name="${mimic_joint_name}">
+        <param name="mimic">${actuated_joint_name}</param>
+        <param name="multiplier">${multiplier}</param>
+        <param name="offset">0</param>
+        <!-- Interfaces are handled automatically on Gazebo and Hardware -->
+      </joint>
+    </xacro:macro>
   <xacro:macro name="ros2_control_robotiq_85_gripper" params="name reduction" >
     <joint name="${name}_finger_joint">
@@ -20,52 +28,22 @@
       <state_interface name="effort" />
     </joint>
-    <joint name="${name}_right_outer_knuckle_joint">
-      <param name="mimic">${name}_finger_joint</param>
-      <param name="multiplier">1</param>
-      <command_interface name="position"/>
-      <state_interface name="position"/>
-      <state_interface name="velocity"/>
-      <state_interface name="effort"/>
-    </joint>
-    <joint name="${name}_right_inner_knuckle_joint">
-      <param name="mimic">${name}_finger_joint</param>
-      <param name="multiplier">1</param>
-      <command_interface name="position"/>
-      <state_interface name="position"/>
-      <state_interface name="velocity"/>
-      <state_interface name="effort"/>
-    </joint>
-    <joint name="${name}_right_inner_finger_joint">
-      <param name="mimic">${name}_finger_joint</param>
-      <param name="multiplier">-1</param>
-      <command_interface name="position"/>
-      <state_interface name="position"/>
-      <state_interface name="velocity"/>
-      <state_interface name="effort"/>
-    </joint>
-    <joint name="${name}_left_inner_finger_joint">
-      <param name="mimic">${name}_finger_joint</param>
-      <param name="multiplier">-1</param>
-      <command_interface name="position"/>
-      <state_interface name="position"/>
-      <state_interface name="velocity"/>
-      <state_interface name="effort"/>
-    </joint>
-    <joint name="${name}_left_inner_knuckle_joint">
-      <param name="mimic">${name}_finger_joint</param>
-      <param name="multiplier">1</param>
-      <command_interface name="position"/>
-      <state_interface name="position"/>
-      <state_interface name="velocity"/>
-      <state_interface name="effort"/>
-    </joint>
-    <joint name="${name}_left_outer_knuckle_joint">
-      <param name="mimic">${name}_finger_joint</param>
-      <param name="multiplier">1</param>
-      <command_interface name="position"/>
-      <state_interface name="position"/>
-      <state_interface name="velocity"/>
-      <state_interface name="effort"/>
-    </joint>
+    <xacro:ros2_control_mimic_joint mimic_joint_name="${name}_right_outer_knuckle_joint"
+                                    actuated_joint_name="${name}_finger_joint"
+                                    multiplier="1"/>
+   <xacro:ros2_control_mimic_joint mimic_joint_name="${name}_right_inner_knuckle_joint"
+                                    actuated_joint_name="${name}_finger_joint"
+                                    multiplier="1"/>
+    <xacro:ros2_control_mimic_joint mimic_joint_name="${name}_right_inner_finger_joint"
+                                    actuated_joint_name="${name}_finger_joint"
+                                    multiplier="-1"/>
+    <xacro:ros2_control_mimic_joint mimic_joint_name="${name}_left_inner_finger_joint"
+                                    actuated_joint_name="${name}_finger_joint"
+                                    multiplier="-1"/>
+    <xacro:ros2_control_mimic_joint mimic_joint_name="${name}_left_inner_knuckle_joint"
+                                    actuated_joint_name="${name}_finger_joint"
+                                    multiplier="-1"/>
+    <xacro:ros2_control_mimic_joint mimic_joint_name="${name}_left_outer_knuckle_joint"
+                                    actuated_joint_name="${name}_finger_joint"
+                                    multiplier="1"/>
     <xacro:include filename="$(find pal_robotiq_description)/urdf/robotiq.transmission.xacro" />
     <xacro:robotiq_transmission prefix="${name}_finger" reduction="${reduction}" />
@@ -78,64 +56,24 @@
       <state_interface name="effort" />
     </joint>
-    <joint name="${name}_right_outer_knuckle_joint">
-      <param name="mimic">${name}_finger_joint</param>
-      <param name="multiplier">-1</param>
-      <command_interface name="position"/>
-      <state_interface name="position"/>
-      <state_interface name="velocity"/>
-      <state_interface name="effort"/>
-    </joint>
-    <joint name="${name}_right_inner_knuckle_joint">
-      <param name="mimic">${name}_finger_joint</param>
-      <param name="multiplier">-1</param>
-      <command_interface name="position"/>
-      <state_interface name="position"/>
-      <state_interface name="velocity"/>
-      <state_interface name="effort"/>
-    </joint>
-    <joint name="${name}_right_inner_finger_joint">
-      <param name="mimic">${name}_finger_joint</param>
-      <param name="multiplier">1</param>
-      <command_interface name="position"/>
-      <state_interface name="position"/>
-      <state_interface name="velocity"/>
-      <state_interface name="effort"/>
-    </joint>
-    <joint name="${name}_left_inner_finger_joint">
-      <param name="mimic">${name}_finger_joint</param>
-      <param name="multiplier">1</param>
-      <command_interface name="position"/>
-      <state_interface name="position"/>
-      <state_interface name="velocity"/>
-      <state_interface name="effort"/>
-    </joint>
-    <joint name="${name}_left_inner_knuckle_joint">
-      <param name="mimic">${name}_finger_joint</param>
-      <param name="multiplier">-1</param>
-      <command_interface name="position"/>
-      <state_interface name="position"/>
-      <state_interface name="velocity"/>
-      <state_interface name="effort"/>
-    </joint>
-    <joint name="${name}_left_outer_knuckle_joint">
-      <param name="mimic">${name}_finger_joint</param>
-      <param name="multiplier">1</param>
-      <command_interface name="position"/>
-      <state_interface name="position"/>
-      <state_interface name="velocity"/>
-      <state_interface name="effort"/>
-    </joint>
+    <xacro:ros2_control_mimic_joint mimic_joint_name="${name}_right_outer_knuckle_joint"
+                                    actuated_joint_name="${name}_finger_joint"
+                                    multiplier="-1"/>
+    <xacro:ros2_control_mimic_joint mimic_joint_name="${name}_right_inner_knuckle_joint"
+                                    actuated_joint_name="${name}_finger_joint"
+                                    multiplier="-1"/>
+    <xacro:ros2_control_mimic_joint mimic_joint_name="${name}_right_inner_finger_joint"
+                                    actuated_joint_name="${name}_finger_joint"
+                                    multiplier="1"/>
+    <xacro:ros2_control_mimic_joint mimic_joint_name="${name}_left_inner_finger_joint"
+                                    actuated_joint_name="${name}_finger_joint"
+                                    multiplier="1"/>
+    <xacro:ros2_control_mimic_joint mimic_joint_name="${name}_left_inner_knuckle_joint"
+                                    actuated_joint_name="${name}_finger_joint"
+                                    multiplier="-1"/>
+    <xacro:ros2_control_mimic_joint mimic_joint_name="${name}_left_outer_knuckle_joint"
+                                    actuated_joint_name="${name}_finger_joint"
+                                    multiplier="1"/>
     <xacro:include filename="$(find pal_robotiq_description)/urdf/robotiq.transmission.xacro" />
     <xacro:robotiq_transmission prefix="${name}_finger" reduction="${reduction}" />
   </xacro:macro>
-  <!-- <xacro:macro name="ros2_control_robotiq_epick" params="name reduction" >
-    <joint name="${name}_joint">
-      <command_interface name="effort" />
-      <state_interface name="position" />
-      <state_interface name="velocity" />
-      <state_interface name="effort" />
-    </joint>
-    <xacro:include filename="$(find pal_robotiq_description)/urdf/robotiq.transmission.xacro" />
-    <xacro:robotiq_transmission name="${name}" reduction="${reduction}" />
-  </xacro:macro> -->
 </robot>

File: pal_robotiq_description/urdf/robotiq_85_gripper.urdf.xacro (robot description, xacro)
@@ -317,4 +317,20 @@
     <xacro:inner_knuckle prefix="${prefix}" fingerprefix="${fingerprefix}" reflect="${reflect}"/>
   </xacro:macro>
+    <!--Dummy joint/link to prevent error with mimic joint
+    See https://github.com/ros-controls/gazebo_ros2_control/issues/173
+    -->
+ <xacro:macro name="dummy_mimic_joint" params="name parent">
+    <link name="${name}_dummy_mimic_link"/>
+    <joint name="${name}_joint_mimic" type="fixed">
+      <parent link="${parent}" />
+      <child link="${name}_dummy_mimic_link" />
+    </joint>
+  </xacro:macro>
+  <xacro:macro name="finger_mimic_dummy" params="prefix fingerprefix">
+    <xacro:dummy_mimic_joint name="${prefix}${fingerprefix}_outer_finger" parent="${prefix}base_link"/>
+    <xacro:dummy_mimic_joint name="${prefix}${fingerprefix}_inner_finger" parent="${prefix}base_link"/>
+    <xacro:dummy_mimic_joint name="${prefix}${fingerprefix}_inner_finger_pad" parent="${prefix}base_link"/>
+    <xacro:dummy_mimic_joint name="${prefix}${fingerprefix}_inner_knuckle" parent="${prefix}base_link"/>
+  </xacro:macro>
   <xacro:macro name="finger_joint" params="prefix">
     <joint name="${prefix}finger_joint" type="revolute">
@@ -351,4 +367,6 @@
     <xacro:finger_links prefix="${prefix}" fingerprefix="left" reflect="1"/>
     <xacro:finger_links prefix="${prefix}" fingerprefix="right" reflect="-1"/>
+    <xacro:finger_mimic_dummy prefix="${prefix}" fingerprefix="left"/>
+    <xacro:finger_mimic_dummy prefix="${prefix}" fingerprefix="right"/>
     <xacro:robotiq_base_joint prefix="${prefix}" />
     <xacro:pal_robotiq_coupling_joint prefix="${prefix}" parent="${parent}">
@@ -357,4 +375,5 @@
     <xacro:finger_joint prefix="${prefix}"/>
     <xacro:right_outer_knuckle_joint prefix="${prefix}"/>
+    <xacro:dummy_mimic_joint name="${prefix}right_outer_knuckle" parent="${prefix}base_link"/>
     <!--This xacro is used to be able to grasp object in simulmation more robustly, it could cause segfault at grasping time -->
     <xacro:gazebo_gripper_grasp name="${prefix}grasp" name_prefix_left="${prefix}left_inner_finger" name_prefix_right="${prefix}right_inner_finger" parent_joint="${parent}"/>
